File: schematics/Gimbal/Gimbal.sch (KiCad schematic (older format))
At the start: 3 parts, among them U1 SN754410, U2 SN754410, U3 SN754410

Commit message: Add working USART code for firmware
Parts:
- added U?: STM32F103C8Tx, Package_QFP:LQFP-48_7x7mm_P0.5mm, symbol MCU_ST_STM32F1:STM32F103C8Tx
- U1, U2, U3: symbol SN754410:SN754410 -> Gimbal-rescue:SN754410-SN754410
Changed lines of the file:
@@
 EESchema Schematic File Version 4
+LIBS:Gimbal-cache
 EELAYER 30 0
 EELAYER END
@@
 $EndDescr
 $Comp
-L SN754410:SN754410 U1
+L Gimbal-rescue:SN754410-SN754410 U1
 U 1 1 5D977634
-P 1900 1600
-F 0 "U1" H 1700 2050 50  0000 C CNN
-F 1 "SN754410" H 1900 1050 50  0000 C CNN
-F 2 "" H 2200 1400 50  0001 C CNN
-F 3 "" H 2200 1400 50  0001 C CNN
-	1    1900 1600
+P 2484 2609
+F 0 "U1" H 2284 3059 50  0000 C CNN
+F 1 "SN754410" H 2484 2059 50  0000 C CNN
+F 2 "" H 2784 2409 50  0001 C CNN
+F 3 "" H 2784 2409 50  0001 C CNN
+	1    2484 2609
 	1    0    0    -1
 $EndComp
 $Comp
-L SN754410:SN754410 U2
+L Gimbal-rescue:SN754410-SN754410 U2
 U 1 1 5D979E75
-P 3300 1600
-F 0 "U2" H 3100 2050 50  0000 C CNN
-F 1 "SN754410" H 3300 1050 50  0000 C CNN
-F 2 "" H 3600 1400 50  0001 C CNN
-F 3 "" H 3600 1400 50  0001 C CNN
-	1    3300 1600
+P 3892 2601
+F 0 "U2" H 3692 3051 50  0000 C CNN
+F 1 "SN754410" H 3892 2051 50  0000 C CNN
+F 2 "" H 4192 2401 50  0001 C CNN
+F 3 "" H 4192 2401 50  0001 C CNN
+	1    3892 2601
 	1    0    0    -1
 $EndComp
 $Comp
-L SN754410:SN754410 U3
+L Gimbal-rescue:SN754410-SN754410 U3
 U 1 1 5D97B113
-P 4850 1600
-F 0 "U3" H 4650 2050 50  0000 C CNN
-F 1 "SN754410" H 4850 1050 50  0000 C CNN
-F 2 "" H 5150 1400 50  0001 C CNN
-F 3 "" H 5150 1400 50  0001 C CNN
-	1    4850 1600
+P 5426 2559
+F 0 "U3" H 5226 3009 50  0000 C CNN
+F 1 "SN754410" H 5426 2009 50  0000 C CNN
+F 2 "" H 5726 2359 50  0001 C CNN
+F 3 "" H 5726 2359 50  0001 C CNN
+	1    5426 2559
 	1    0    0    -1
 $EndComp
+$Comp
+L MCU_ST_STM32F1:STM32F103C8Tx U?
+U 1 1 5D9765E6
+P 7098 2464
+F 0 "U?" H 7048 875 50  0000 C CNN
+F 1 "STM32F103C8Tx" H 7048 784 50  0000 C CNN
+F 2 "Package_QFP:LQFP-48_7x7mm_P0.5mm" H 6498 1064 50  0001 R CNN
+F 3 "http://www.st.com/st-web-ui/static/active/en/resource/technical/document/datasheet/CD00161566.pdf" H 7098 2464 50  0001 C CNN
+	1    7098 2464
+	1    0    0    -1
+$EndComp
